Commit message: mppi

File: urdf/robot.urdf (robot description, URDF)
Before this commit: robot mecanum_car, 5 links, 4 joints
Joints:
- joint base_joint: origin xyz=0 0 0 rpy=0 0 0 -> xyz=0 0 0.07 rpy=0 0 0
- joint front_indicator_joint: origin xyz=0.1 0 0.04 rpy=0 0 0 -> xyz=0.0915 0 0.08 rpy=0 0 0
- joint lidar_joint: origin xyz=0.05 0 0.14 rpy=0 0 1.5708 -> xyz=0.05 0 0.14 rpy=0 0 -1.5708
